File: Hardware/RFID_GPS_BOARD/RFID_GPS_BOARD.sch (KiCad schematic (older format))
At the start: 13 parts, among them J1 GPS_Module_Coonector, J2 Barrel_Jack_Switch, U1 RC522_RFID, U2 NodeMCU_1.0_(ESP-12E), U3 L7805, U4 I2c_LCD

Commit message: completed project final
Parts:
- removed C?: .1uF, Capacitor_THT:C_Disc_D3.0mm_W1.6mm_P2.50mm, symbol Device:C_Small
Changed lines of the file:
@@
 	2250 1400 2250 1500
 Connection ~ 2250 1500
-$Comp
-L Device:C_Small C?
-U 1 1 5CFA432B
-P 6450 2900
-F 0 "C?" H 6542 2946 50  0000 L CNN
-F 1 ".1uF" H 6542 2855 50  0000 L CNN
-F 2 "Capacitor_THT:C_Disc_D3.0mm_W1.6mm_P2.50mm" H 6450 2900 50  0001 C CNN
-F 3 "~" H 6450 2900 50  0001 C CNN
-	1    6450 2900
-	1    0    0    -1
-$EndComp
-$Comp
-L power:+5V #PWR?
-U 1 1 5CFA4332
-P 6700 2700
-F 0 "#PWR?" H 6700 2550 50  0001 C CNN
-F 1 "+5V" H 6715 2873 50  0000 C CNN
-F 2 "" H 6700 2700 50  0001 C CNN
-F 3 "" H 6700 2700 50  0001 C CNN
-	1    6700 2700
-	1    0    0    -1
-$EndComp
-$Comp
-L power:GND #PWR?
-U 1 1 5CFA4338
-P 6700 3050
-F 0 "#PWR?" H 6700 2800 50  0001 C CNN
-F 1 "GND" H 6705 2877 50  0000 C CNN
-F 2 "" H 6700 3050 50  0001 C CNN
-F 3 "" H 6700 3050 50  0001 C CNN
-	1    6700 3050
-	1    0    0    -1
-$EndComp
-Wire Wire Line
-	6450 3000 6700 3000
-Wire Wire Line
-	6450 2800 6700 2800
-Wire Wire Line
-	6700 2700 6700 2800
-Wire Wire Line
-	6700 3050 6700 3000
 $EndSCHEMATC
